File: 32Vin_3.3Vout_Regulator.kicad_sch (KiCad schematic)
At the start: 8 parts, among them J1 PinSocket_1x04_P2.54mm_Vertic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, U1 AP63203WU

Commit message: MPN and feeder updated for the chip
Parts:
- U1: Feeder (none) -> 8mm; MPN (none) -> C780769
Changed lines of the file:
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@@
+			)
+		)
+		(property "MPN" "C780769"
+			(at 85.09 35.56 0)
+			(effects
+				(font
+					(size 1.27 1.27)
+				)
+				(hide yes)
+			)
+		)
+		(property "Feeder" "8mm"
+			(at 85.09 35.56 0)
+			(effects
+				(font
+					(size 1.27 1.27)
+				)
+				(hide yes)
 			)
 		)
