File: panel.kicad_pcb (KiCad board)
At the start: 2 copper layers, 48.2 x 68.9 mm, 93 parts, among them J1 PinSocket_1x04_P2.54mm_Vertic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, U1 AP63203WU

Commit message: Reduce screw hole size to match M2
Parts:
- J1 (x9): value PinSocket_1x04_P2.54mm_Vertical_SMD_Pin1Left -> Regulator
- turned KiKit_FID_B_1 to 180 degrees
- turned KiKit_FID_B_2 to 180 degrees
- turned KiKit_FID_B_3 to 180 degrees
- turned KiKit_FID_B_4 to 180 degrees
Other:
- outline, holes or cut-outs redrawn
